File: BreadboardPowerSupply_v2/BreadboardPowerSupply_v2.kicad_sch (KiCad schematic)
At the start: 15 parts, among them J1 Barrel_Jack_Switch, J2 Conn_02x02_Odd_Even, J3 Conn_02x02_Odd_Even, SW1 SW_DPDT_x2, U1 LM7805_TO220

Commit message: Added LED
Parts:
- added D?: LED, LED_THT:LED_D5.0mm, symbol Device:LED
Connections:
- net V-: now also D?.1 (K)
- net Vout1: now also D?.2 (A)
Changed lines of the file:
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@@
   (junction (at 105.41 121.92) (diameter 0) (color 0 0 0 0)
   )
+  (junction (at 125.984 121.92) (diameter 0) (color 0 0 0 0)
+  )
   (junction (at 83.82 106.68) (diameter 0) (color 0 0 0 0)
   )
@@
   )
   (junction (at 204.47 98.425) (diameter 0) (color 0 0 0 0)
+  )
+  (junction (at 125.984 93.345) (diameter 0) (color 0 0 0 0)
   )
   (junction (at 72.39 104.14) (diameter 0) (color 0 0 0 0)
@@
     (stroke (width 0) (type default) (color 0 0 0 0))
   )
+  (wire (pts (xy 115.57 121.92) (xy 125.984 121.92))
+    (stroke (width 0) (type default) (color 0 0 0 0))
+  )
   (wire (pts (xy 201.295 90.805) (xy 201.295 83.185))
     (stroke (width 0) (type default) (color 0 0 0 0))
@@
     (stroke (width 0) (type default) (color 0 0 0 0))
   )
-  (wire (pts (xy 115.57 121.92) (xy 134.62 121.92))
-    (stroke (width 0) (type default) (color 0 0 0 0))
-  )
   (wire (pts (xy 134.62 121.92) (xy 151.765 121.92))
     (stroke (width 0) (type default) (color 0 0 0 0))
@@
     (stroke (width 0) (type default) (color 0 0 0 0))
   )
+  (wire (pts (xy 125.984 93.345) (xy 134.62 93.345))
+    (stroke (width 0) (type default) (color 0 0 0 0))
+  )
   (polyline (pts (xy 92.71 78.105) (xy 92.71 127))
     (stroke (width 0) (type default) (color 0 0 0 0))
@@
     (stroke (width 0) (type default) (color 0 0 0 0))
   )
+  (wire (pts (xy 125.984 112.776) (xy 125.984 121.92))
+    (stroke (width 0) (type default) (color 0 0 0 0))
+  )
   (wire (pts (xy 225.425 90.805) (xy 219.71 90.805))
     (stroke (width 0) (type default) (color 0 0 0 0))
   )
-  (wire (pts (xy 123.19 93.345) (xy 134.62 93.345))
+  (wire (pts (xy 123.19 93.345) (xy 125.984 93.345))
     (stroke (width 0) (type default) (color 0 0 0 0))
   )
@@
     (stroke (width 0) (type default) (color 0 0 0 0))
   )
+  (wire (pts (xy 125.984 121.92) (xy 134.62 121.92))
+    (stroke (width 0) (type default) (color 0 0 0 0))
+  )
   (wire (pts (xy 151.765 97.79) (xy 151.765 93.345))
+    (stroke (width 0) (type default) (color 0 0 0 0))
+  )
+  (wire (pts (xy 125.984 93.345) (xy 125.984 105.156))
     (stroke (width 0) (type default) (color 0 0 0 0))
   )
@@
     (pin "2")
   )
+  (symbol (lib_id "Device:LED") (at 125.984 108.966 90) (unit 1)
+    (in_bom yes) (on_board yes) (fields_autoplaced)
+    (property "Reference" "D?" (id 0) (at 129.794 109.2834 90)
+      (effects (font (size 1.27 1.27)) (justify right))
+    )
+    (property "Value" "LED" (id 1) (at 129.794 111.8234 90)
+      (effects (font (size 1.27 1.27)) (justify right))
+    )
+    (property "Footprint" "LED_THT:LED_D5.0mm" (id 2) (at 125.984 108.966 0)
+      (effects (font (size 1.27 1.27)) hide)
+    )
+    (property "Datasheet" "~" (id 3) (at 125.984 108.966 0)
+      (effects (font (size 1.27 1.27)) hide)
+    )
+    (pin "1")
+    (pin "2")
+  )
   (symbol (lib_id "Device:LED") (at 151.765 113.665 90) (unit 1)
     (in_bom yes) (on_board yes) (fields_autoplaced)
@@
       (reference "D6") (unit 1) (value "LED") (footprint "LED_THT:LED_D5.0mm")
     )
+    (path "/5ce23b6b-bd8c-44d9-a91a-04985175beda"
+      (reference "D?") (unit 1) (value "LED") (footprint "LED_THT:LED_D5.0mm")
+    )
     (path "/dccf9fb7-59df-4e02-baa6-536501382604"

Commit message: Added net label
Connections:
- net Vout1 renamed LED_REGULADOR
Changed lines of the file:
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@@
     (effects (font (size 1.27 1.27)) (justify left bottom))
+  )
+  (label "LED_REGULADOR" (at 125.984 102.87 180)
+    (effects (font (size 1.27 1.27)) (justify right bottom))
   )
   (label "Vout1" (at 142.875 93.345 0)
